Commit message: Add IK-driven pick-and-place; fix detachable-joint init
demo_sequence.py only replayed hand-picked joint angles and never approached the
object - it moved, it did not pick. pick_and_place.py replaces it: every arm pose
is solved by inverse kinematics from the target's measured TF pose.

- Chain: FK, Jacobian and damped-least-squares IK parsed straight from the URDF,
  so no MoveIt config is needed to reach a Cartesian goal.
- IK solves position exactly, then ranks solutions by how closely the achieved
  gripper approach matches the requested one. A hard top-down constraint is
  unsatisfiable here: with four joints limited to 0..pi the most downward
  approach reachable over the panel is ~53 degrees off vertical, so demanding
  [0,0,-1] failed every solve even though the point is exactly reachable.
- object_tf_publisher.py broadcasts named object frames. ros_gz_bridge's
  Pose_V -> TFMessage conversion leaves frame ids EMPTY on Jazzy and the
  PoseArray conversion drops names, so neither can identify one object.
- DetachableJoint named parent_link "gripper_palm", which does not exist in the
  converted SDF: sdformat merges fixed-joint-connected links into their parent,
  folding tool0/gripper_palm/grasp_link into link6. The plugin aborted at startup
  and /gripper/attach silently did nothing.
- world_to_base now carries the 0.5 m pedestal height and the model spawns at
  z=0, so TF and Gazebo agree; previously every TF-derived goal was 0.5 m out.
- kill_sim.sh: orphaned servers corrupt recordings and block controllers. It
  spares its own ancestors, since a caller's command line usually matches the
  kill pattern and a naive pgrep kills the invoking shell.

Grasp retention across the full transfer is still intermittent - see the summary
in the next commit's notes.

Co-Authored-By: Claude Opus 5 <noreply@anthropic.com>

File: panda_ws/src/uw_arm_description/urdf/uw_arm.gazebo.xacro (robot description, xacro)
@@ -122,5 +122,15 @@
         <plugin filename="gz-sim-detachable-joint-system"
                 name="gz::sim::systems::DetachableJoint">
-          <parent_link>gripper_palm</parent_link>
+          <!-- link6, NOT gripper_palm. sdformat merges every link joined by a
+               FIXED joint into its parent, so tool0, gripper_palm and grasp_link
+               do not exist as links in the converted SDF - they are all folded
+               into link6. Naming gripper_palm here makes the plugin abort at
+               startup with
+                 [Err] [DetachableJoint.cc:62] Link with name [gripper_palm]
+                 not found in model [uw_arm]
+               and, because the failure is only a log line, /gripper/attach then
+               silently does nothing: the object is held by jaw friction alone
+               and drops or is left behind mid-transfer. -->
+          <parent_link>link6</parent_link>
           <child_model>${model}</child_model>
           <child_link>${link}</child_link>

File: panda_ws/src/uw_arm_description/urdf/uw_arm.urdf.xacro (robot description, xacro)
@@ -109,7 +109,13 @@
   <!-- ==================================================================== -->
   <link name="world"/>
+  <!-- The pedestal height lives HERE, and the model is spawned at z=0, so TF and
+       Gazebo agree on where the robot is. Spawning at z=0.5 against an identity
+       joint instead leaves robot_state_publisher placing base_link at world z=0
+       while physics has it at 0.5: every TF-derived target is then half a metre
+       out and IK cannot converge on it. -->
+  <xacro:property name="base_mount_z" value="0.5"/>
   <joint name="world_to_base" type="fixed">
     <parent link="world"/><child link="base_link"/>
-    <origin xyz="0 0 0" rpy="0 0 0"/>
+    <origin xyz="0 0 ${base_mount_z}" rpy="0 0 0"/>
   </joint>
   <!-- ==================================================================== -->
