Commit message: Fix gripper actuation, jaw geometry and payload trim
Four defects found by measurement, each independently enough to break a grasp:

1. Only one finger was ever actuated. gz_ros2_control does not mirror URDF
   <mimic> joints - finger_right_joint never moved and never even appeared in
   /joint_states, so the gripper closed one-sided and shoved the object away.
   Both fingers are now independently commanded by a JointTrajectoryController
   (GripperActionController drives exactly one joint, so it could not be used).

2. DetachableJoint never latched. gz-sim 8.11 ignores <attach_topic>: with
   suppress_initial_attach the joint is never created and /gripper/attach does
   nothing, though the plugin loads and subscribes. Verified by publishing attach
   and driving the arm away with the target left sitting on the panel. Removed.

3. Jaw-face geometry was wrong by 6 mm per side. The finger joint sits at
   half_gap=0.012 but the finger box is 0.012 thick, so the inner face is at
   0.006+q, not 0.012+q. The commanded "3 mm squeeze" was really 9 mm of
   penetration, which the contact solver resolves by ejecting the object.
   Measured payload displacement fell from 0.127 m to 0.035 m when the nominal
   squeeze was doubled - the opposite of the intent.

4. Payload was 4.14 N net-negative (density 2000). Real intervention cargo is
   trimmed near neutral; the canister is now ~1100 kg/m^3 for 0.32 N net.

Also: IK now rejects solutions whose jaw axis is not near horizontal, since the
jaws cannot close across the canister's 120 mm height, only its 60 mm width.

Arm-side control is exact - commanded vs achieved grasp pose measures 0.7 mm.
Grasp retention through the transfer is still not reliable; see the notes in the
next message.

Co-Authored-By: Claude Opus 5 <noreply@anthropic.com>

File: panda_ws/src/uw_arm_description/urdf/gripper.xacro (robot description, xacro)
@@ -66,6 +66,11 @@
       <dynamics damping="2.0" friction="0.5"/>
     </joint>
-    <!-- Passive follower. ros2_control (Jazzy) reads this <mimic> tag directly,
-         so finger_right must NOT appear in the <ros2_control> block. -->
+    <!-- Both jaws are INDEPENDENTLY ACTUATED and commanded together by the
+         gripper controller. This deliberately does NOT use a <mimic> tag:
+         gz_ros2_control does not mirror URDF mimic joints here, so the right
+         finger never moved and never even appeared in /joint_states. The gripper
+         then closed with one jaw only, shoving the object sideways instead of
+         gripping it - the single cause behind grasps that "closed" and still
+         left the payload behind. -->
     <joint name="finger_right_joint" type="prismatic">
       <parent link="gripper_palm"/><child link="finger_right"/>
@@ -74,5 +79,4 @@
       <limit lower="0.0" upper="${stroke}" effort="60" velocity="0.1"/>
       <dynamics damping="2.0" friction="0.5"/>
-      <mimic joint="finger_left_joint" multiplier="1.0" offset="0.0"/>
     </joint>
     <!-- Grasp target frame: mid-way up the jaws, on the approach axis.

File: panda_ws/src/uw_arm_description/urdf/uw_arm.gazebo.xacro (robot description, xacro)
@@ -105,8 +105,8 @@
     <!-- ================================================================== -->
     <gazebo reference="finger_left">
-      <mu1>1.6</mu1><mu2>1.6</mu2><kp>1e6</kp><kd>50.0</kd><minDepth>0.001</minDepth>
+      <mu1>3.0</mu1><mu2>3.0</mu2><kp>1e6</kp><kd>50.0</kd><minDepth>0.001</minDepth>
     </gazebo>
     <gazebo reference="finger_right">
-      <mu1>1.6</mu1><mu2>1.6</mu2><kp>1e6</kp><kd>50.0</kd><minDepth>0.001</minDepth>
+      <mu1>3.0</mu1><mu2>3.0</mu2><kp>1e6</kp><kd>50.0</kd><minDepth>0.001</minDepth>
     </gazebo>
     <!-- ================================================================== -->
@@ -142,5 +142,17 @@
       </gazebo>
     </xacro:macro>
-    <xacro:graspable model="target_canister"/>
+    <!-- NOT INSTANTIATED. gz-sim 8.11's DetachableJoint does not honour
+         <attach_topic>: with <suppress_initial_attach>true</suppress_initial_attach>
+         the joint is never created, and publishing /gripper/attach silently does
+         nothing even though the plugin loads and subscribes. Verified directly -
+         after publishing attach and driving the arm away, the target stayed put.
+         The grasp is carried by jaw friction instead, which the numbers support
+         comfortably: the canister weighs 8.48 N and displaces 4.34 N, so 4.14 N
+         net must be held; with mu=2.0 across two jaws that needs about 1.0 N of
+         normal force per jaw. What was actually breaking grasps was the gripper
+         closing one-sided (see gripper.xacro), not a shortage of friction.
+         Re-enable this if you move to a Gazebo version whose DetachableJoint
+         supports re-attaching:
+             <xacro:graspable model="target_canister"/> -->
     <!-- ================================================================== -->
     <!--  WRIST RGB-D SENSOR                                                 -->

File: panda_ws/src/uw_arm_description/urdf/uw_arm.ros2_control.xacro (robot description, xacro)
@@ -32,14 +32,22 @@
       <xacro:arm_ji name="joint5" init="0.0"/>
       <xacro:arm_ji name="joint6" init="1.5708"/>
+      <!-- BOTH fingers are commanded. There is no mimic joint: gz_ros2_control
+           does not mirror URDF <mimic> here, which left the right jaw frozen and
+           absent from /joint_states, so the gripper closed one-sided and pushed
+           objects away instead of gripping them. -->
       <xacro:if value="${use_gripper}">
-        <joint name="finger_left_joint">
-          <command_interface name="position">
-            <param name="min">0.0</param>
-            <param name="max">0.035</param>
-          </command_interface>
-          <state_interface name="position"><param name="initial_value">0.035</param></state_interface>
-          <state_interface name="velocity"/>
-          <state_interface name="effort"/>
-        </joint>
+        <xacro:macro name="finger_ji" params="name">
+          <joint name="${name}">
+            <command_interface name="position">
+              <param name="min">0.0</param>
+              <param name="max">0.035</param>
+            </command_interface>
+            <state_interface name="position"><param name="initial_value">0.035</param></state_interface>
+            <state_interface name="velocity"/>
+            <state_interface name="effort"/>
+          </joint>
+        </xacro:macro>
+        <xacro:finger_ji name="finger_left_joint"/>
+        <xacro:finger_ji name="finger_right_joint"/>
       </xacro:if>
     </ros2_control>
